File: PROJECT-OVERDRIVE.kicad_pcb (KiCad board)
At the start: 2 copper layers, 225 parts, among them J1 PJ-327A0-SMT, J2 USB_C_Receptacle_USB2.0_16P, K1 G6S-2, Q1 AO3400A, Q10 AO3400A, Q2 AO3400A, Q3 AO3400A, Q4 AO3400A, Q5 AO3400A, Q6 AO3400A, Q7 AO3400A, Q8 AO3400A, Q9 AO3400A, U1 CH32V30xVxTx, U2 PCM5102APWR, U3 MAX4410EUD+, Y1 Crystal

Commit message: idkmyinternetwasdead.git
Parts:
- removed D10, D100, D101, D102, D103, D104, D105, D106, D107, D108, D109, D11, D110, D111, D112, D113, D114, D115, D116, D117, D118, D119, D12, D120, D121, D122, D123, D124, D125, D126, D127, D128, D129, D13, D130, D131, D132, D133, D134, D135, D136, D137, D138, D139, D14, D140, D141, D142, D143, D144, D145, D146, D147, D148, D149, D15, D150, D151, D152, D153, D154, D155, D156, D157, D158, D159, D16, D160, D17, D18, D19, D2, D20, D21, D22, D23, D24, D25, D26, D27, D28, D29, D3, D30, D31, D32, D33, D34, D35, D36, D37, D38, D39, D4, D40, D41, D42, D43, D44, D45, D46, D47, D48, D49, D5, D50, D51, D52, D53, D54, D55, D56, D57, D58, D59, D6, D60, D61, D62, D63, D64, D65, D66, D67, D68, D69, D7, D70, D71, D72, D73, D74, D75, D76, D77, D78, D79, D8, D80, D81, D82, D83, D84, D85, D86, D87, D88, D89, D9, D90, D91, D92, D93, D94, D95, D96, D97, D98, D99: LED_45deg, LED_SMD:LED_0805_2012Metric
- added C14: 1u, Capacitor_SMD:C_0603_1608Metric, F.Cu at (148.7, 143.7)
- added C15: 1u, Capacitor_SMD:C_0603_1608Metric, F.Cu at (148.7, 146.2)
- added C16: 0.1u, Capacitor_SMD:C_0603_1608Metric, F.Cu at (148.7, 148.7)
- added C17: 0.1u, Capacitor_SMD:C_0603_1608Metric, F.Cu at (148.7, 151.2)
- added C18: 0.1u, Capacitor_SMD:C_0603_1608Metric, F.Cu at (148.7, 153.7)
- added C19: 4.7u, Capacitor_SMD:C_0603_1608Metric, F.Cu at (148.7, 156.2)
- added C20: 4.7u, Capacitor_SMD:C_0603_1608Metric, F.Cu at (148.7, 158.7)
- added C21: 0.1u, Capacitor_SMD:C_0603_1608Metric, F.Cu at (152.7, 143.7)
- added C22: 2.2u, Capacitor_SMD:C_0603_1608Metric, F.Cu at (152.7, 146.2)
- added C23: 4.7u, Capacitor_SMD:C_0603_1608Metric, F.Cu at (152.7, 148.7)
- added C24: 4.7u, Capacitor_SMD:C_0603_1608Metric, F.Cu at (152.7, 151.2)
- added C25: 4.7u, Capacitor_SMD:C_0603_1608Metric, F.Cu at (152.7, 153.7)
- added C26: 0.1u, Capacitor_SMD:C_0603_1608Metric, F.Cu at (152.7, 156.2)
- added C27: 0.1u, Capacitor_SMD:C_0603_1608Metric, F.Cu at (152.7, 158.7)
- added C28: 4.7u, Capacitor_SMD:C_0603_1608Metric, F.Cu at (156.7, 143.7)
- added C29: 4.7u, Capacitor_SMD:C_0603_1608Metric, F.Cu at (156.7, 146.2)
- added C30: 4.7u, Capacitor_SMD:C_0805_2012Metric, F.Cu at (165.3, 161.6)
- added C31: 4.7u, Capacitor_SMD:C_0805_2012Metric, F.Cu at (165.3, 164.6)
- added C32: 0.1u, Capacitor_SMD:C_0805_2012Metric, F.Cu at (165.3, 167.6)
- added C33: 0.1u, Capacitor_SMD:C_0805_2012Metric, F.Cu at (169.8, 161.6)
- added C34: 4.7u, Capacitor_SMD:C_0805_2012Metric, F.Cu at (169.8, 164.6)
- added C35: 0.1u, Capacitor_SMD:C_0805_2012Metric, F.Cu at (169.8, 167.6)
- added C36: 4.7u, Capacitor_SMD:C_0805_2012Metric, F.Cu at (174.2, 161.6)
- added C37: 4.7u, Capacitor_SMD:C_0805_2012Metric, F.Cu at (174.2, 164.6)
- added C38: 0.1u, Capacitor_SMD:C_0805_2012Metric, F.Cu at (174.2, 167.6)
- added F1: 200ma, Fuse:Fuse_0805_2012Metric, F.Cu at (160.9, 143.9)
- added F2: 100ma, Fuse:Fuse_0805_2012Metric, F.Cu at (160.9, 146.8)
- added F3: 250ma, Fuse:Fuse_0805_2012Metric, F.Cu at (160.9, 149.8)
- added F4: 250ma, Fuse:Fuse_0805_2012Metric, F.Cu at (160.9, 152.7)
- added JP2: SolderJumper_3_Bridged12, Jumper:SolderJumper-3_P1.3mm_Bridged12_RoundedPad1.0x1.5mm, F.Cu at (170.7, 144.2)
- added JP3: SolderJumper_3_Bridged12, Jumper:SolderJumper-3_P1.3mm_Bridged12_RoundedPad1.0x1.5mm, F.Cu at (170.7, 148.0)
- added JP4: SolderJumper_3_Bridged12, Jumper:SolderJumper-3_P1.3mm_Bridged12_RoundedPad1.0x1.5mm, F.Cu at (170.7, 151.8)
- added Q1: AO3401A, Package_TO_SOT_SMD:SOT-23, F.Cu at (149.1, 162.4)
- added Q2: AO3401A, Package_TO_SOT_SMD:SOT-23, F.Cu at (149.1, 167.0)
- added Q3: S8050, Package_TO_SOT_THT:TO-92_Inline, F.Cu at (153.5, 163.2)
- added R10: 1k, Resistor_SMD:R_0805_2012Metric_Pad1.20x1.40mm_HandSolder, F.Cu at (165.5, 152.7)
- added R11: 10k, Resistor_SMD:R_0805_2012Metric_Pad1.20x1.40mm_HandSolder, F.Cu at (165.5, 155.7)
- added R12: 10k, Resistor_SMD:R_0805_2012Metric_Pad1.20x1.40mm_HandSolder, F.Cu at (165.5, 158.6)
- added R13: 22r, Resistor_SMD:R_0603_1608Metric, F.Cu at (156.7, 148.7)
- added R14: 22r, Resistor_SMD:R_0603_1608Metric, F.Cu at (156.7, 151.2)
- added R15: 22r, Resistor_SMD:R_0603_1608Metric, F.Cu at (156.7, 153.7)
- added R16: 1k, Resistor_SMD:R_0805_2012Metric, F.Cu at (160.9, 161.6)
- added R5: 22k, Resistor_SMD:R_0805_2012Metric_Pad1.20x1.40mm_HandSolder, F.Cu at (165.5, 143.9)
- added R6: 22k, Resistor_SMD:R_0805_2012Metric_Pad1.20x1.40mm_HandSolder, F.Cu at (165.5, 146.8)
- added R7: 10k, Resistor_SMD:R_0805_2012Metric, F.Cu at (160.9, 155.7)
- added R8: 100k, Resistor_SMD:R_0805_2012Metric, F.Cu at (160.9, 158.6)
- added R9: 1k, Resistor_SMD:R_0805_2012Metric_Pad1.20x1.40mm_HandSolder, F.Cu at (165.5, 149.8)
- added RN2: 22, Resistor_SMD:R_Array_Concave_4x0603, F.Cu at (153.6, 168.2)
- added U4: AP2112K-3.3, Package_TO_SOT_SMD:SOT-23-5, F.Cu at (176.1, 144.8)
- added U5: AP2112K-3.3, Package_TO_SOT_SMD:SOT-23-5, F.Cu at (176.1, 149.4)
- C1: value C -> 2.2u; footprint Capacitor_SMD:C_0805_2012Metric_Pad1.18x1.45mm_HandSolder -> Capacitor_SMD:C_0603_1608Metric
- D1: value LED_45deg -> SS34; footprint LED_SMD:LED_0805_2012Metric -> Diode_SMD:D_SMA
- R33, R34: value 22k -> 10k
- Y1: value Crystal -> 8M
- moved D1 64.8 mm to (171.9, 156.2)
Connections:
- D1 pad 2: Net-(D1-A) -> VBUS
- J1 pad 2: unconnected-(J1-Pad2) -> Net-(J1-Pad2)
- J1 pad 3: unconnected-(J1-Pad3) -> GND
- J1 pad 4: unconnected-(J1-Pad4) -> GND
- J1 pad 5: unconnected-(J1-Pad5) -> Net-(J1-Pad5)
- J1 pad 6: unconnected-(J1-Pad6) -> Net-(U6A--)
- J2 pad A4: Net-(J2-VBUS-PadA4) -> VBUS
- J2 pad A9: Net-(J2-VBUS-PadA4) -> VBUS
- J2 pad B4: Net-(J2-VBUS-PadA4) -> VBUS
- J2 pad B9: Net-(J2-VBUS-PadA4) -> VBUS
- K1 pad 1: unconnected-(K1-Pad1) -> +5V
- K1 pad 12: unconnected-(K1-Pad12) -> Net-(Q3-C)
- K1 pad 4: unconnected-(K1-Pad4) -> Net-(J1-Pad5)
- K1 pad 9: unconnected-(K1-Pad9) -> Net-(J1-Pad2)
- U1 pad 47: unconnected-(U1-PB10-Pad47) -> I2C_SCL
- U1 pad 48: unconnected-(U1-PB11-Pad48) -> I2C_SDA
- U1 pad 51: unconnected-(U1-PB12-Pad51) -> Net-(RN2-R4.1)
- U1 pad 52: unconnected-(U1-PB13-Pad52) -> Net-(RN2-R3.1)
- U1 pad 53: unconnected-(U1-PB14-Pad53) -> Net-(RN2-R2.1)
- U1 pad 54: unconnected-(U1-PB15-Pad54) -> Net-(RN2-R1.1)
- U1 pad 77: unconnected-(U1-PA15-Pad77) -> Net-(U1-PA15)
- U1 pad 89: unconnected-(U1-PB3-Pad89) -> Net-(U1-PB3)
- U1 pad 91: unconnected-(U1-PB5-Pad91) -> Net-(U1-PB5)
- U1 pad 97: unconnected-(U1-PE0-Pad97) -> Net-(U1-PE0)
- U1 pad 98: unconnected-(U1-PE1-Pad98) -> Net-(U1-PE1)
- U2 pad 1: +3.3VA -> +3.3VDAC
- U2 pad 10: unconnected-(U2-DEMP-Pad10) -> Net-(JP3-C)
- U2 pad 11: unconnected-(U2-FLT-Pad11) -> Net-(JP4-C)
- U2 pad 12: unconnected-(U2-SCK-Pad12) -> GND
- U2 pad 13: unconnected-(U2-BCK-Pad13) -> DAC_BCK
- U2 pad 14: unconnected-(U2-DIN-Pad14) -> DAC_DIN
- U2 pad 15: unconnected-(U2-LRCK-Pad15) -> DAC_LRCLK
- U2 pad 16: unconnected-(U2-FMT-Pad16) -> Net-(JP2-C)
- U2 pad 17: unconnected-(U2-XSMT-Pad17) -> DAC_MUTE
- U2 pad 18: unconnected-(U2-LDOO-Pad18) -> Net-(U2-LDOO)
- U2 pad 19: unconnected-(U2-DGND-Pad19) -> GND
- U2 pad 2: unconnected-(U2-CAPP-Pad2) -> Net-(U2-CAPP)
- U2 pad 20: unconnected-(U2-DVDD-Pad20) -> VDDF
- U2 pad 3: unconnected-(U2-CPGND-Pad3) -> GND
- U2 pad 4: unconnected-(U2-CAPM-Pad4) -> Net-(U2-CAPM)
- U2 pad 5: unconnected-(U2-VNEG-Pad5) -> Net-(U2-VNEG)
- U2 pad 8: unconnected-(U2-AVDD-Pad8) -> +3.3VDAC
- U2 pad 9: unconnected-(U2-AGND-Pad9) -> GND
- U3 pad 1: unconnected-(U3-*SHDNL-Pad1) -> AMP_MUTE
- U3 pad 12: unconnected-(U3-*SHDNR-Pad12) -> AMP_MUTE
- U3 pad 6: unconnected-(U3-PVSS-Pad6) -> Net-(U3-PVSS)
- U3 pad 7: unconnected-(U3-SVSS-Pad7) -> Net-(U3-PVSS)
